File: auto_gardener.brd (EAGLE design)
At the start: 83.1 x 55.1 mm, 38 parts, among them IC4 LM2596S

Commit message: Update design to version 1.0
Parts:
- removed L3: 100uH, SparkFun-Passives:INDUCTOR_SDR1307
- added L1: 100uH/3A, inductor-sumida:CDRH127/LD
- IC4: value LM2596S -> LM2576
- moved IC4 9.83 mm to (44.3, 29.6)
- moved OLED 8.13 mm to (35.9, 33.7)
- moved R1 5.67 mm to (70.4, 27.6), turned to 0 degrees
- moved U$8 4.99 mm to (58.3, 33.5)
- moved N4148 4.21 mm to (65.9, 29.1)
- moved C1815 3.94 mm to (66.7, 23.9)
- moved R4 3.75 mm to (75.6, 27.6), turned to 0 degrees
- moved D2 2.80 mm to (73.7, 23.9)
- moved R3 2.33 mm to (70.4, 30.2), turned to 180 degrees
- moved U$2 1.14 mm to (79.5, 51.4)
- moved R5 1.09 mm to (75.6, 30.4), turned to 0 degrees
- moved U$6 0.90 mm to (79.4, 2.67)
- moved LED1 0.77 mm to (79.9, 24.9)
- moved LED2 0.77 mm to (79.9, 30.9)
- moved X1 0.38 mm to (75.6, 13.2)
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Connections:
- net +3V3: now also SW_BTN.1; no longer SW_BTN.3
- net 5V: now also L1.2; no longer L3.P$2
- net D3: now also OLED.4; no longer OLED.3
- net D4: now also OLED.3; no longer OLED.4
- net D8: now also SW_BTN.3; no longer SW_BTN.1
- net N$9: now also L1.1; no longer L3.P$1
Routing:
- net GND: track 282.9 -> 245.8 mm, vias 2 -> 1
- net A5: track 33.6 -> 58.4 mm
- net D6: track 56.8 -> 40.2 mm, vias 0 -> 1
- net A2: track 41.3 -> 56.1 mm
- net 5V: track 184.1 -> 169.5 mm, vias 3 -> 2
- net D8: track 89.7 -> 76.7 mm
- net A3: track 44.1 -> 56.2 mm, vias 0 -> 2
- net D3: track 31.3 -> 22.1 mm
- net D4: track 34.9 -> 26.3 mm
- net +3V3: track 126.3 -> 133.9 mm
- net VIN: track 75.6 -> 68.8 mm
- net D7: track 47.8 -> 41.6 mm
- net A7: track 21.2 -> 26.8 mm, vias 0 -> 2
- net N$3: track 9.47 -> 3.95 mm
- net A0: track 39.3 -> 44.8 mm, vias 0 -> 1
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Other:
- board size 83.1 x 55.1 mm -> 82.2 x 55.1 mm
- board text added: "Auto Gardener v1"
- board text removed: "Auto Gardener v0.2"
