File: auto_gardener.sch (EAGLE design)
At the start: 34 parts, among them IC4 LM2596S

Commit message: Update design to version 1.0
Parts:
- removed L3: 100uH, SparkFun-Passives:INDUCTORSDR13-7-270ML
- added L1: 100uH/3A, inductor-sumida:CDRH127/LD
- IC4: value LM2596S -> LM2576
Connections:
- net +3V3: now also SW_BTN.1; no longer SW_BTN.2
- net 5V: now also L1.2; no longer L3.2
- net D3: now also OLED.4; no longer OLED.3
- net D4: now also OLED.3; no longer OLED.4
- net D8: now also SW_BTN.2; no longer SW_BTN.1
- net N$9: now also L1.1; no longer L3.1
Other:
- note added: "File:"
- moved on the sheet: A1, A2, A3, A4, A5, A6, A7, A8, C1815, C5, C6, CAP_BTN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
